File: pcb-files/main-digital/weerstation-main.kicad_sch (KiCad schematic)
At the start: 29 parts, among them J1 sds011 pm10 pm2.5 dust sensor, J10 PCA9685 servo controller, J16 analoog bord connector, J2 analoog bord connector (digit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, J23 temp sensor AM2315C, J24 veml 7700, J25 VL53L0X, J26 hc-sr04, J28 regenmeter digitaal flip sens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, J29 mpu-9265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

Commit message: update pcb files better layout and grounding inproved
Parts:
- added H1, H10, H11, H12, H2, H3, H4, H5, H6, H7, H8, H9: MountingHole, MountingHole:MountingHole_long, symbol Mechanical:MountingHole
